Commit message: turned joint torso to head into fixed

File: urdf/actuators/head.urdf.xacro (robot description, xacro)
@@ -53,5 +53,5 @@
       </visual>
     </link>
-    <joint name="joint_${parent}_to_${name}" type="revolute">
+    <joint name="joint_${parent}_to_${name}" type="fixed">
       <origin xyz="-0.06 0 ${(pole_size_z/2)+(head_base_length)+(head_box_size_z/2)}" rpy="0 0 0"/>
       <child link="${name}"/>
