Commit message: Added simple transmissions and hardware interfaces to each joint of urdf

File: urdf/actuators/manipulator/manip.urdf.xacro (robot description, xacro)
@@ -2,4 +2,16 @@
 <robot xmlns:xacro="http://www.ros.org/wiki/xacro" name="hera_description">
 <xacro:include filename="$(find hera_description)/urdf/actuators/manipulator/manip_prop.urdf.xacro"/>
+  <xacro:macro name="SimpleTransmission" params="joint">
+    <transmission name="transmission_${joint}">
+      <type>transmission_interface/SimpleTransmission</type>
+      <joint name="${joint}">
+        <hardwareInterface>hardware_interface/PositionJointInterface</hardwareInterface>
+      </joint>
+        <actuator name="motor_${joint}">
+            <hardwareInterface>hardware_interface/PositionJointInterface</hardwareInterface>
+            <mechanicalReduction>1</mechanicalReduction>
+        </actuator>
+    </transmission>
+  </xacro:macro>
 <!--manip_base_link-->
   <xacro:macro name="create_manip_base_link">
@@ -58,4 +70,5 @@
       <limit lower="-1.57" upper="1.57" effort="0" velocity="5" />
     </joint>
+    <xacro:SimpleTransmission joint="shoulder_pan_joint"/>
   </xacro:macro>
 <!--link_2: shoulder_lift_link-->
@@ -87,4 +100,5 @@
       <limit lower="-0.9" upper="3.55" effort="0" velocity="5" />
     </joint>
+    <xacro:SimpleTransmission joint="shoulder_lift_joint"/>
   </xacro:macro>
 <!--link_3: elbow_pan_link-->
@@ -116,4 +130,5 @@
       <limit lower="-0.8" upper="0.8" effort="0" velocity="5" />
     </joint>
+    <xacro:SimpleTransmission joint="elbow_pan_joint"/>
   </xacro:macro>
 <!--link_4: elbow_lift_link-->
@@ -145,4 +160,5 @@
       <limit lower="-3.55" upper="0.9" effort="0" velocity="5" />
     </joint>
+    <xacro:SimpleTransmission joint="elbow_lift_joint"/>
   </xacro:macro>
 <!--link_5: wrist_pan_link-->
@@ -174,4 +190,5 @@
       <limit lower="-3.14" upper="3.14" effort="0" velocity="5" />
     </joint>
+    <xacro:SimpleTransmission joint="wrist_pan_joint"/>
   </xacro:macro>
 <!--link_6: wrist_lift_link-->
@@ -203,4 +220,5 @@
       <limit lower="-0.64" upper="4" effort="0" velocity="5" />
     </joint>
+    <xacro:SimpleTransmission joint="wrist_lift_joint"/>
   </xacro:macro>
 <!--link_7: gripper_right_link-->
@@ -232,4 +250,5 @@
       <limit lower="-0.6454" upper="1.5600" effort="0" velocity="5" />
     </joint>
+    <xacro:SimpleTransmission joint="gripper_right_joint"/>
   </xacro:macro>
 <!--link_7_end: gripper_right_end_link-->

Commit message: deleted simulation gripper

File: urdf/actuators/manipulator/manip.urdf.xacro (robot description, xacro)
@@ -128,5 +128,5 @@
       <child link="elbow_pan_link" />
       <axis xyz="1 0 0" />
-      <limit lower="-0.8" upper="0.8" effort="0" velocity="5" />
+      <limit lower="-1.57" upper="1.57" effort="0" velocity="5" />
     </joint>
     <xacro:SimpleTransmission joint="elbow_pan_joint"/>
@@ -188,5 +188,5 @@
       <child link="wrist_pan_link" />
       <axis xyz="1 0 0" />
-      <limit lower="-3.14" upper="3.14" effort="0" velocity="5" />
+      <limit lower="-1.57" upper="3.14" effort="0" velocity="5" />
     </joint>
     <xacro:SimpleTransmission joint="wrist_pan_joint"/>

Commit message: changed gripper's close limits

File: urdf/actuators/manipulator/manip.urdf.xacro (robot description, xacro)
@@ -248,5 +248,5 @@
       <child  link="gripper_right_link" />
       <axis xyz="0 0 1" />
-      <limit lower="-0.6454" upper="1.5600" effort="0" velocity="5" />
+      <limit lower="-0.8" upper="0.0" effort="0" velocity="5" />
     </joint>
     <xacro:SimpleTransmission joint="gripper_right_joint"/>
@@ -306,5 +306,5 @@
       <child link="gripper_left_link" />
       <axis xyz="0 0 1" />
-      <limit lower="-1.5600" upper="0.6454" effort="0" velocity="5" />
+      <limit lower="0.0" upper="0.8" effort="0" velocity="5" />
     </joint>
   </xacro:macro>

Commit message: increased wrist pan's limits

File: urdf/actuators/manipulator/manip.urdf.xacro (robot description, xacro)
@@ -188,5 +188,5 @@
       <child link="wrist_pan_link" />
       <axis xyz="1 0 0" />
-      <limit lower="-1.57" upper="3.14" effort="0" velocity="5" />
+      <limit lower="-3.14" upper="3.14" effort="0" velocity="5" />
     </joint>
     <xacro:SimpleTransmission joint="wrist_pan_joint"/>

Commit message: increased gripper's lower limit

File: urdf/actuators/manipulator/manip.urdf.xacro (robot description, xacro)
@@ -248,5 +248,5 @@
       <child  link="gripper_right_link" />
       <axis xyz="0 0 1" />
-      <limit lower="-0.8" upper="0.0" effort="0" velocity="5" />
+      <limit lower="-1.0" upper="0.0" effort="0" velocity="5" />
     </joint>
     <xacro:SimpleTransmission joint="gripper_right_joint"/>
@@ -306,5 +306,5 @@
       <child link="gripper_left_link" />
       <axis xyz="0 0 1" />
-      <limit lower="0.0" upper="0.8" effort="0" velocity="5" />
+      <limit lower="0.0" upper="1.0" effort="0" velocity="5" />
     </joint>
   </xacro:macro>

Commit message: inverted manip's pose

File: urdf/actuators/manipulator/manip.urdf.xacro (robot description, xacro)
@@ -35,5 +35,5 @@
   <!--manip_base_joint-->
     <joint name="manip_base_joint" type="fixed">
-      <origin xyz="0.27075 0 0.0295" rpy="0 0 0" />
+      <origin xyz="0.27075 0 0.0295" rpy="3.14 0 0" />
       <parent link="manip_support_link" />
       <child link="manip_base_link" />
