Commit message: added zed2 to description

File: robots/hera_full.urdf.xacro (robot description, xacro)
@@ -20,5 +20,6 @@
   <xacro:include filename="$(find hera_description)/urdf/sensors/hokuyo_urg.urdf.xacro"/>
   <xacro:include filename="$(find hera_description)/urdf/sensors/asus_xtion.urdf.xacro"/>
-  <xacro:include filename="$(find hera_description)/urdf/sensors/kinect_one.urdf.xacro"/>
+  <!-- <xacro:include filename="$(find hera_description)/urdf/sensors/kinect_one.urdf.xacro"/> -->
+  <xacro:include filename="$(find hera_description)/urdf/sensors/zed.urdf.xacro" />
   <!-- simulation -->
   <xacro:include filename="$(find hera_description)/urdf/simulation/colors.gazebo.xacro" />
@@ -63,9 +64,14 @@
   </xacro:xtion>
   <!-- torso pointcloud front: kinect_one -->
-  <xacro:kinect_one
+  <!-- <xacro:kinect_one
     name="kinect_one"
     parent="torso_sensor_plat">
     <origin xyz="0.05 0 0.1" rpy="0 0 0" />
-  </xacro:kinect_one>
+  </xacro:kinect_one> -->
+  <!-- torso pointcloud front: zed2 -->
+  <xacro:zed_camera name="zed2" model="zed2" parent="torso_sensor_plat">
+    <origin xyz="0.0 0.0 0.0" rpy="0.0 0.0 0.0" />
+  </xacro:zed_camera>
+  <link name="base_link" />
   <!--torso suporte-->
   <xacro:create_manip_support_link
@@ -103,4 +109,8 @@
     reference="kinect_one"
     update_rate="30"/>
+  <!-- zed2 -->
+  <xacro:gazebo_zed2
+    reference="zed2"
+    update_rate="30"/>
   <xacro:manip_transmission/>
 </robot>

File: urdf/commons.urdf.xacro (robot description, xacro)
@@ -18,4 +18,7 @@
   <material name="white">
     <color rgba="1.0 1.0 1.0 1.0"/>
+  </material>
+  <material name="zed2_mat">
+      <color rgba="0.25 0.25 0.25 0.99"/>
   </material>
   <!-- Macros -->

Commit message: added zed2 to description completed

File: robots/hera_full.urdf.xacro (robot description, xacro)
@@ -28,5 +28,6 @@
   <xacro:include filename="$(find hera_description)/urdf/simulation/hokuyo_urg.gazebo.xacro" />
   <xacro:include filename="$(find hera_description)/urdf/simulation/asus_xtion.gazebo.xacro" />
-  <xacro:include filename="$(find hera_description)/urdf/simulation/kinect_one.gazebo.xacro" />
+  <!-- <xacro:include filename="$(find hera_description)/urdf/simulation/kinect_one.gazebo.xacro" /> -->
+  <xacro:include filename="$(find hera_description)/urdf/simulation/zed2.gazebo.xacro" />
   <xacro:include filename="$(find hera_description)/urdf/simulation/manipulator.gazebo.xacro" />
   <xacro:include filename="$(find hera_description)/urdf/simulation/control.gazebo.xacro" />
@@ -70,8 +71,7 @@
   </xacro:kinect_one> -->
   <!-- torso pointcloud front: zed2 -->
-  <xacro:zed_camera name="zed2" model="zed2" parent="torso_sensor_plat">
-    <origin xyz="0.0 0.0 0.0" rpy="0.0 0.0 0.0" />
+  <xacro:zed_camera name="zed" model="zed2" parent="torso_sensor_plat">
+    <origin xyz="0.015 0 0.085" rpy="0 0 0" />
   </xacro:zed_camera>
-  <link name="base_link" />
   <!--torso suporte-->
   <xacro:create_manip_support_link
@@ -106,7 +106,7 @@
     update_rate="30"/>
   <!-- kinect_one -->
-  <xacro:gazebo_kinect_one
+  <!-- <xacro:gazebo_kinect_one
     reference="kinect_one"
-    update_rate="30"/>
+    update_rate="30"/> -->
   <!-- zed2 -->
   <xacro:gazebo_zed2

File: urdf/commons.urdf.xacro (robot description, xacro)
@@ -18,7 +18,4 @@
   <material name="white">
     <color rgba="1.0 1.0 1.0 1.0"/>
-  </material>
-  <material name="zed2_mat">
-      <color rgba="0.25 0.25 0.25 0.99"/>
   </material>
   <!-- Macros -->

File: urdf/sensors/zed.urdf.xacro (robot description, xacro)
@@ -16,5 +16,4 @@
 -->
 <robot xmlns:xacro="http://wiki.ros.org/xacro">
-  <xacro:include filename="$(find hera_description/urdf/commons.urdf.xacro" />
   <xacro:property name="M_PI"     value="3.1415926535897931" />
   <!--
@@ -47,5 +46,5 @@
           <mesh filename="package://hera_description/meshes/zed2.stl" />
         </geometry>
-        <material name="${model}_mat" />
+        <material name="black" />
       </visual>
       <collision>

Commit message: added option to choose kinect or zed

File: robots/hera_full.urdf.xacro (robot description, xacro)
@@ -17,8 +17,9 @@
   <xacro:include filename="$(find hera_description)/urdf/actuators/manipulator/manip.urdf.xacro" />
   <!-- sensors -->
+  <xacro:property name="camera" value="zed"/> <!-- choose kinect or zed-->
   <xacro:include filename="$(find hera_description)/urdf/sensors/hokuyo_utm.urdf.xacro"/>
   <xacro:include filename="$(find hera_description)/urdf/sensors/hokuyo_urg.urdf.xacro"/>
   <xacro:include filename="$(find hera_description)/urdf/sensors/asus_xtion.urdf.xacro"/>
-  <!-- <xacro:include filename="$(find hera_description)/urdf/sensors/kinect_one.urdf.xacro"/> -->
+  <xacro:include filename="$(find hera_description)/urdf/sensors/kinect_one.urdf.xacro"/>
   <xacro:include filename="$(find hera_description)/urdf/sensors/zed.urdf.xacro" />
   <!-- simulation -->
@@ -28,5 +29,5 @@
   <xacro:include filename="$(find hera_description)/urdf/simulation/hokuyo_urg.gazebo.xacro" />
   <xacro:include filename="$(find hera_description)/urdf/simulation/asus_xtion.gazebo.xacro" />
-  <!-- <xacro:include filename="$(find hera_description)/urdf/simulation/kinect_one.gazebo.xacro" /> -->
+  <xacro:include filename="$(find hera_description)/urdf/simulation/kinect_one.gazebo.xacro" />
   <xacro:include filename="$(find hera_description)/urdf/simulation/zed2.gazebo.xacro" />
   <xacro:include filename="$(find hera_description)/urdf/simulation/manipulator.gazebo.xacro" />
@@ -64,14 +65,18 @@
     <origin xyz="0.215 0 -0.17" rpy="0 0 0" />
   </xacro:xtion>
-  <!-- torso pointcloud front: kinect_one -->
-  <!-- <xacro:kinect_one
-    name="kinect_one"
-    parent="torso_sensor_plat">
-    <origin xyz="0.05 0 0.1" rpy="0 0 0" />
-  </xacro:kinect_one> -->
-  <!-- torso pointcloud front: zed2 -->
-  <xacro:zed_camera name="zed" model="zed2" parent="torso_sensor_plat">
-    <origin xyz="0.015 0 0.085" rpy="0 0 0" />
-  </xacro:zed_camera>
+  <!-- kinect -->
+  <xacro:if value="${camera == 'kinect'}">
+    <xacro:kinect_one
+      name="kinect_one"
+      parent="torso_sensor_plat">
+      <origin xyz="0.05 0 0.1" rpy="0 0 0" />
+    </xacro:kinect_one>
+  </xacro:if>
+  <!-- zed -->
+  <xacro:if value="${camera == 'zed'}">
+    <xacro:zed_camera name="zed" model="zed2" parent="torso_sensor_plat">
+      <origin xyz="0.015 0 0.085" rpy="0 0 0" />
+    </xacro:zed_camera>
+  </xacro:if>
   <!--torso suporte-->
   <xacro:create_manip_support_link

Commit message: Changed position of xtion camera and removed kinect/zed

File: robots/hera_full.urdf.xacro (robot description, xacro)
@@ -62,9 +62,9 @@
   <xacro:xtion
     name="xtion_link"
-    parent="torso">
-    <origin xyz="0.215 0 -0.17" rpy="0 0 0" />
+    parent="torso_sensor_plat">
+    <origin xyz="0.05 0 0.0" rpy="0 0 0" />
   </xacro:xtion>
   <!-- kinect -->
-  <xacro:if value="${camera == 'kinect'}">
+  <!--xacro:if value="${camera == 'kinect'}">
     <xacro:kinect_one
       name="kinect_one"
@@ -72,5 +72,5 @@
       <origin xyz="0.05 0 0.1" rpy="0 0 0" />
     </xacro:kinect_one>
-  </xacro:if>
+  </xacro:if-->
   <!-- zed -->
   <!-- <xacro:if value="${camera == 'zed'}">

Commit message: Calibration of xtion position

File: robots/hera_full.urdf.xacro (robot description, xacro)
@@ -63,5 +63,5 @@
     name="xtion_link"
     parent="torso_sensor_plat">
-    <origin xyz="0.05 0 0.0" rpy="0 0 0" />
+    <origin xyz="0.02 0 0.05" rpy="0 0 0" />
   </xacro:xtion>
   <!-- kinect -->

Commit message: Simulation description

File: robots/hera_full.urdf.xacro (robot description, xacro)
@@ -48,18 +48,18 @@
     parent="torso"/>
   <!-- base laser front -->
-  <xacro:hokuyo_utm
+  <xacro:hokuyo_urg
     name="base_scan_front"
     parent="base">
-    <origin xyz="0.3 0 0.01" rpy="0 0 0"/>
-  </xacro:hokuyo_utm>
+    <origin xyz="0.3 0 0.08" rpy="0 0 0"/>
+  </xacro:hokuyo_urg>
   <!-- base laser back -->
-  <xacro:hokuyo_urg
+  <!-- <xacro:hokuyo_urg
     name="base_scan_back"
     parent="base">
-    <origin xyz="-0.3 0 0.01" rpy="0 0 ${M_PI}"/>
-  </xacro:hokuyo_urg>
+    <origin xyz="-0.3 0 0.06" rpy="0 0 ${M_PI}"/>
+  </xacro:hokuyo_urg> -->
   <!-- torso pointcloud front: xtion -->
   <xacro:xtion
-    name="camera_link"
+    name="xtion"
     parent="torso_sensor_plat">
     <origin xyz="0.02 0 0.05" rpy="0 0 0" />
@@ -86,5 +86,5 @@
     parent="torso"/>
   <!-- manip -->
-  <xacro:manipulator/>
+  <!-- <xacro:manipulator/> -->
 <!-- ####################################################################### -->
 <!-- ####################### gazebo extensions ##############################-->

File: urdf/actuators/torso.urdf.xacro (robot description, xacro)
@@ -101,5 +101,5 @@
       <child link="${name}"/>
     </joint>
-    <joint name="joint_${name}_to_${name}_sensor_plat" type="revolute">
+    <joint name="joint_${name}_to_${name}_sensor_plat" type="fixed">
       <origin xyz="0.09 0 0.46" rpy="0 0 0"/>
       <parent link="${name}"/>

File: urdf/simulation/hokuyo_utm.gazebo.xacro (robot description, xacro)
@@ -18,5 +18,5 @@
           <range>
 	          <min>0.08</min>
-	          <max>30.0</max>
+	          <max>5.0</max>
 	          <resolution>0.01</resolution>
           </range>

Commit message: Added new head motors and torso (missing joints and camera_link)

File: robots/hera_full.urdf.xacro (robot description, xacro)
@@ -17,5 +17,5 @@
   <xacro:include filename="$(find hera_description)/urdf/actuators/manipulator/manip.urdf.xacro" />
   <!-- sensors -->
-  <xacro:property name="camera" value="zed"/> <!-- choose kinect or zed-->
+  // <xacro:property name="camera" value="zed"/> <!-- choose kinect or zed-->
   <xacro:include filename="$(find hera_description)/urdf/sensors/hokuyo_utm.urdf.xacro"/>
   <xacro:include filename="$(find hera_description)/urdf/sensors/hokuyo_urg.urdf.xacro"/>
@@ -59,10 +59,4 @@
     <origin xyz="-0.3 0 0.01" rpy="0 0 ${M_PI}"/>
   </xacro:hokuyo_urg>
-  <!-- torso pointcloud front: xtion -->
-  <xacro:xtion
-    name="camera_link"
-    parent="torso_sensor_plat">
-    <origin xyz="0.02 0 0.05" rpy="0 0 0" />
-  </xacro:xtion>
   <!-- kinect -->
   <!--xacro:if value="${camera == 'kinect'}">

File: urdf/actuators/torso.urdf.xacro (robot description, xacro)
@@ -29,44 +29,9 @@
     <!-- torso -->
     <link name="${name}">
-      <xacro:create_box
-        m="${big_box_mass}"
-        x="${big_box_size_x}"
-        y="${big_box_size_y}"
-        z="${big_box_size_z}">
-        <origin xyz="-0.1 0 -0.225" rpy="0 0 0"/>
-      </xacro:create_box>
-      <xacro:create_box
-        m="${small_box_mass}"
-        x="${small_box_size_x}"
-        y="${small_box_size_y}"
-        z="${small_box_size_z}">
-        <origin xyz="0.15 0 -0.35" rpy="0 0 0"/>
-      </xacro:create_box>
-      <xacro:create_box
-        m="${head_plat_mass}"
-        x="${head_plat_size_x}"
-        y="${head_plat_size_y}"
-        z="${head_plat_size_z}">
-        <origin xyz="-0.06 0 0.475" rpy="0 0 0"/>
-      </xacro:create_box>
-      <xacro:create_box
-        m="${pole_mass}"
-        x="${pole_size_x}"
-        y="${pole_size_y}"
-        z="${pole_size_z}">
-        <origin xyz="-0.06 -0.18 0" rpy="0 0 0"/>
-      </xacro:create_box>
-      <xacro:create_box
-        m="${pole_mass}"
-        x="${pole_size_x}"
-        y="${pole_size_y}"
-        z="${pole_size_z}">
-        <origin xyz="-0.06 0.18 0" rpy="0 0 0"/>
-      </xacro:create_box>
       <visual>
-        <origin xyz="0 0 -0.5" rpy="0 0 0"/>
+        <origin xyz="0 0 -0.5" rpy="1.57 0 0"/>
         <material name="dark_grey"/>
         <geometry>
-          <mesh filename="package://hera_description/meshes/torso.stl"/>
+          <mesh filename="package://hera_description/meshes/torso.stl" scale="0.001 0.001 0.001"/>
         </geometry>
       </visual>
@@ -79,18 +44,21 @@
       </collision>
     </link>
-    <!-- sensor plat -->
-    <link name="${name}_sensor_plat">
-      <xacro:create_box
-        m="${sensor_plat_mass}"
-        x="${sensor_plat_size_x}"
-        y="${sensor_plat_size_y}"
-        z="${sensor_plat_size_z}">
-        <origin xyz="0 0 0.05" rpy="0 0 0"/>
-      </xacro:create_box>
+    <!-- head_pan -->
+    <link name="camera_pan">
       <visual>
-        <origin xyz="0.2 0 -0.2" rpy="0 0 0"/>
-        <material name="dark_grey"/>
+        <origin xyz="-0.035 -0.02 -0.047" rpy="3.14 1.57 3.14"/>
+        <material name="white"/>
         <geometry>
-          <mesh filename="package://hera_description/meshes/torso_sensor_plat.stl"/>
+          <mesh filename="package://hera_description/meshes/camera_meshes/Intermediario.stl" scale="0.001 0.001 0.001"/>
+        </geometry>
+      </visual>
+    </link>
+    <!-- head_lift -->
+    <link name="camera_lift">
+      <visual>
+        <origin xyz="-0.125 0.02 -0.507" rpy="0 -1.54 -3.14"/>
+        <material name="white"/>
+        <geometry>
+          <mesh filename="package://hera_description/meshes/camera_meshes/Inferior.stl" scale="0.001 0.001 0.001"/>
         </geometry>
       </visual>
@@ -101,18 +69,26 @@
       <child link="${name}"/>
     </joint>
-    <joint name="joint_${name}_to_${name}_sensor_plat" type="revolute">
+    <joint name="joint_camera_pan" type="revolute">
       <origin xyz="0.09 0 0.46" rpy="0 0 0"/>
       <parent link="${name}"/>
-      <child link="${name}_sensor_plat"/>
+      <child link="camera_pan"/>
       <axis xyz="0 1 0"/>
       <limit effort="${torso_sensor_plat_effort}" velocity="${torso_sensor_plat_velocity}"
-        lower="0.0" upper="1.8"/>
+        lower="-0.3" upper="1.5"/>
     </joint>
-    <transmission name="tran_${name}_sensor_plat">
+  <joint name="joint_camera_lift" type="revolute">
+      <origin xyz="0.09 0 0.46" rpy="0 0 0"/>
+      <parent link="camera_pan"/>
+      <child link="camera_lift"/>
+      <axis xyz="0 1 0"/>
+      <limit effort="${torso_sensor_plat_effort}" velocity="${torso_sensor_plat_velocity}"
+        lower="-0.3" upper="1.5"/>
+    </joint>
+    <transmission name="tran_camera_pan">
       <type>transmission_interface/SimpleTransmission</type>
-      <joint name="joint_${name}_to_${name}_sensor_plat">
+      <joint name="joint_${name}_to_camera_pan">
         <hardwareInterface>hardware_interface/EffortJointInterface</hardwareInterface>
       </joint>
-      <actuator name="motor_${name}_sensor_plat">
+      <actuator name="motor_camera_pan">
         <hardwareInterface>hardware_interface/EffortJointInterface</hardwareInterface>
         <mechanicalReduction>1</mechanicalReduction>

Commit message: Add dynamixel.stl and sensor_d435i to hera_full.urdf.xacro

File: robots/hera_full.urdf.xacro (robot description, xacro)
@@ -5,4 +5,5 @@
        xmlns:interface="http://playerstage.sourceforge.net/gazebo/xmlschema/#interface"
        xmlns:xacro="http://ros.org/wiki/xacro">
+    <xacro:arg name="use_nominal_extrinsics" default="false" />
     <xacro:include filename="$(find hera_description)/urdf/utils/utils.xacro.xml"/>
     <xacro:include filename="$(find hera_description)/urdf/base/base.xacro.xml"/>
@@ -22,4 +23,5 @@
     <xacro:include filename="$(find hera_description)/urdf/gazebo/control.xacro.xml" />
     <xacro:include filename="$(find hera_description)/urdf/gazebo/manipulator.xacro.xml" />
+    <xacro:include filename="$(find realsense2_description)/urdf/_d435i.urdf.xacro"/>
     <!-- Robot -->
     <!-- base -->
@@ -41,9 +43,4 @@
     </xacro:hokuyo_urg>
     <!-- torso pointcloud front: xtion -->
-    <xacro:xtion
-        name="xtion"
-        parent="torso_sensor_plat">
-        <origin xyz="0.02 0 0.05" rpy="0 0 0" />
-    </xacro:xtion>
     <!-- manip support-->
     <xacro:create_manip_support_link
@@ -52,4 +49,7 @@
     <xacro:create_backrest_link
         parent="torso"/>
+    <xacro:sensor_d435i parent="torso_pan_mechanism_link" use_nominal_extrinsics="$(arg use_nominal_extrinsics)">
+        <origin xyz="0 0 0" rpy="0 0 0"/>
+    </xacro:sensor_d435i>
     <!--manipulator-->
     <xacro:manipulator/>
@@ -72,8 +72,5 @@
         min_angle="-1.45"
         max_angle="1.45" />
-    <!-- xtion -->
-    <xacro:gazebo_xtion
-        reference="xtion"
-        update_rate="30"/>
-    <xacro:generate_transmission_position joint_name="joint_torso_to_torso_sensor_plat"/>
+    <xacro:generate_transmission_position joint_name="joint_camera_pan"/>
+    <xacro:generate_transmission_position joint_name="joint_camera_tilt"/>
 </robot>

Commit message: Update URDF file to use new Realsense D435 sensor model with Gazebo Plugin

File: robots/hera_full.urdf.xacro (robot description, xacro)
@@ -23,5 +23,5 @@
     <xacro:include filename="$(find hera_description)/urdf/gazebo/control.xacro.xml" />
     <xacro:include filename="$(find hera_description)/urdf/gazebo/manipulator.xacro.xml" />
-    <xacro:include filename="$(find realsense2_description)/urdf/_d435i.urdf.xacro"/>
+    <xacro:include filename="$(find hera_description)/urdf/sensors/realsense_d435.urdf.xacro"/>
     <!-- Robot -->
     <!-- base -->
@@ -49,7 +49,7 @@
     <xacro:create_backrest_link
         parent="torso"/>
-    <xacro:sensor_d435i parent="torso_pan_mechanism_link" use_nominal_extrinsics="$(arg use_nominal_extrinsics)">
-        <origin xyz="0 0 0" rpy="0 0 0"/>
-    </xacro:sensor_d435i>
+    <xacro:sensor_d435 parent="torso_pan_mechanism_link">
+        <origin xyz="0 0 0.03" rpy="0 0 0"/>
+    </xacro:sensor_d435>
     <!--manipulator-->
     <xacro:manipulator/>
